Commit message: pve first try

File: mh5_hardware/urdf/mh5_hardware.xacro (robot description, xacro)
@@ -2,9 +2,30 @@
 <robot xmlns:xacro="http://www.ros.org/wiki/xacro">
   <xacro:macro name="mh5_hardware" params="name use_mock_hardware">
+    <xacro:macro name="register_init" params="name address length value">
+      <param name="init_${name}">${address},${length},${value} </param>
+    </xacro:macro>
+    <xacro:macro name="common_init">
+      <xacro:register_init name="return_delay" address="9" length="1" value="0" />
+      <xacro:register_init name="operating_mode" address="11" length="1" value="3" />
+      <xacro:register_init name="temp_limit" address="31" length="1" value="75" />
+      <xacro:register_init name="volt_limit" address="32" length="2" value="135" />
+      <xacro:register_init name="vel_limit" address="44" length="4" value="1023" />
+      <xacro:register_init name="min_pos" address="52" length="4" value="0" />
+      <xacro:register_init name="max_pos" address="48" length="4" value="4095" />
+    </xacro:macro>
+    <xacro:macro name="mh5_servo" params="joint_name id">
+      <joint name="${joint_name}">
+        <param name="id">${id}</param>
+        <xacro:common_init />
+        <state_interface name="position"/>
+        <state_interface name="velocity"/>
+        <state_interface name="effort"/>
+      </joint>
+    </xacro:macro>
     <ros2_control name="upper_body" type="system">
       <xacro:unless value="${use_mock_hardware}">
         <hardware>
           <plugin>mh5_hardware/MH5DynamixelBus</plugin>
-          <param name="debug">no</param>
+          <param name="debug">yes</param>
           <param name="port">/dev/ttySC0</param>
           <param name="baudrate">2000000</param>
@@ -13,9 +34,14 @@
         </hardware>
       </xacro:unless>
-      <joint name="l_sho_p">
-        <state_interface name="position"/>
-        <state_interface name="velocity"/>
-        <state_interface name="load"/>
-      </joint>
+      <xacro:mh5_servo joint_name="l_sho_p" id="34" />
+      <xacro:mh5_servo joint_name="l_sho_r" id="33" />
+      <xacro:mh5_servo joint_name="l_elb_y" id="32" />
+      <xacro:mh5_servo joint_name="l_elb_p" id="31" />
+      <xacro:mh5_servo joint_name="r_sho_p" id="44" />
+      <xacro:mh5_servo joint_name="r_sho_r" id="43" />
+      <xacro:mh5_servo joint_name="r_elb_y" id="42" />
+      <xacro:mh5_servo joint_name="r_elb_p" id="41" />
+      <xacro:mh5_servo joint_name="head_y" id="51" />
+      <xacro:mh5_servo joint_name="head_p" id="52" />
       <!-- <xacro:if value="${use_mock_hardware}">
         <hardware>

Commit message: pve - working; direction fixed

File: mh5_hardware/urdf/mh5_hardware.xacro (robot description, xacro)
@@ -5,6 +5,7 @@
       <param name="init_${name}">${address},${length},${value} </param>
     </xacro:macro>
-    <xacro:macro name="common_init">
+    <xacro:macro name="common_init" params="direction">
       <xacro:register_init name="return_delay" address="9" length="1" value="0" />
+      <xacro:register_init name="drive_mode" address="10" length="1" value="${direction}" />
       <xacro:register_init name="operating_mode" address="11" length="1" value="3" />
       <xacro:register_init name="temp_limit" address="31" length="1" value="75" />
@@ -14,14 +15,20 @@
       <xacro:register_init name="max_pos" address="48" length="4" value="4095" />
     </xacro:macro>
-    <xacro:macro name="mh5_servo" params="joint_name id">
+    <xacro:macro name="mh5_servo" params="joint_name id direction">
       <joint name="${joint_name}">
         <param name="id">${id}</param>
-        <xacro:common_init />
-        <state_interface name="position"/>
-        <state_interface name="velocity"/>
-        <state_interface name="effort"/>
+        <xacro:common_init direction="${direction}" />
+        <state_interface name="position" />
+        <state_interface name="velocity" />
+        <state_interface name="effort" />
       </joint>
     </xacro:macro>
     <ros2_control name="upper_body" type="system">
+      <xacro:if value="${use_mock_hardware}">
+        <hardware>
+          <plugin>mock_components/GenericSystem</plugin>
+          <param name="calculate_dynamics">true</param>
+        </hardware>
+      </xacro:if>
       <xacro:unless value="${use_mock_hardware}">
         <hardware>
@@ -34,75 +41,19 @@
         </hardware>
       </xacro:unless>
-      <xacro:mh5_servo joint_name="l_sho_p" id="34" />
-      <xacro:mh5_servo joint_name="l_sho_r" id="33" />
-      <xacro:mh5_servo joint_name="l_elb_y" id="32" />
-      <xacro:mh5_servo joint_name="l_elb_p" id="31" />
-      <xacro:mh5_servo joint_name="r_sho_p" id="44" />
-      <xacro:mh5_servo joint_name="r_sho_r" id="43" />
-      <xacro:mh5_servo joint_name="r_elb_y" id="42" />
-      <xacro:mh5_servo joint_name="r_elb_p" id="41" />
-      <xacro:mh5_servo joint_name="head_y" id="51" />
-      <xacro:mh5_servo joint_name="head_p" id="52" />
-      <!-- <xacro:if value="${use_mock_hardware}">
-        <hardware>
-          <plugin>mock_components/GenericSystem</plugin>
-          <param name="calculate_dynamics">true</param>
-        </hardware>
-      </xacro:if> -->
-      <!-- <xacro:macro name="wheel_joint" params="side pin_p pin_n">
-        <joint name="${side}_wheel_joint">
-          <command_interface name="velocity"/>
-          <command_interface name="max_velocity"/>
-          <state_interface name="velocity"/>
-          <param name="pin_p">${pin_p}</param>
-          <param name="pin_n">${pin_n}</param>
-          <param name="model">MotorHBridgeNoecoder</param>
-          <param name="max_velocity">19.8962</param>
-        </joint>
-      </xacro:macro> -->
-      <!-- <xacro:macro name="button" params="id">
-        <gpio name="button_${id}">
-          <state_interface name="pressed"/>
-          <state_interface name="led"/>
-          <command_interface name="reset"/>
-          <command_interface name="led"/>
-        </gpio>
-      </xacro:macro> -->
-      <!-- <xacro:macro name="rgb_led" params="id">
-        <gpio name="led_${id}">
-          <command_interface name="red"/>
-          <command_interface name="green"/>
-          <command_interface name="blue"/>
-        </gpio>
-      </xacro:macro> -->
-<!--
-      <xacro:wheel_joint side="left" pin_p="11" pin_n="8" />
-      <xacro:wheel_joint side="right" pin_p="10" pin_n="9" />       -->
-      <!-- <sensor name="ultrasonic">
-        <command_interface name="offset">
-          <param name="initial_value">190000</param>
-          <param name="min">10000</param>
-          <param name="max">500000</param>
-        </command_interface>
-        <command_interface name="timeout">
-          <param name="initial_value">50</param>
-        </command_interface>
-        <command_interface name="samples">
-          <param name="initial_value">10</param>
-        </command_interface>
-        <state_interface name="distance"/>
-        <param name="pin_trigger">13</param>
-        <param name="pin_echo">25</param>
-      </sensor> -->
-      <!-- <xacro:button id="a" />
-      <xacro:button id="b" />
-      <xacro:button id="x" />
-      <xacro:button id="y" /> -->
-      <!-- <xacro:rgb_led id="front_left" />
-      <xacro:rgb_led id="front_right" />
-      <xacro:rgb_led id="middle_left" />
-      <xacro:rgb_led id="middle_right" />
-      <xacro:rgb_led id="back_left" />
-      <xacro:rgb_led id="back_right" /> -->
+      <xacro:mh5_servo joint_name="l_sho_p" id="34" direction="1" />
+      <xacro:mh5_servo joint_name="l_sho_r" id="33" direction="1" />
+      <xacro:mh5_servo joint_name="l_elb_y" id="32" direction="1" />
+      <xacro:mh5_servo joint_name="l_elb_p" id="31" direction="0" />
+      <xacro:mh5_servo joint_name="r_sho_p" id="44" direction="0" />
+      <xacro:mh5_servo joint_name="r_sho_r" id="43" direction="0" />
+      <xacro:mh5_servo joint_name="r_elb_y" id="42" direction="0" />
+      <xacro:mh5_servo joint_name="r_elb_p" id="41" direction="1" />
+      <xacro:mh5_servo joint_name="head_p" id="51" direction="0" />
+      <xacro:mh5_servo joint_name="head_y" id="52" direction="0" />
+      <sensor name="pve_communication">
+        <param name="rate">200</param>
+        <state_interface name="packets" />
+        <state_interface name="errors" />
+      </sensor>
     </ros2_control>
     <!-- <ros2_control name="imu" type="sensor">

Commit message: - support for XL330 servos in URDF - added the grippers - include offset handling for knee servos - fixed handling of status read at different frequency - take advantage of async scheduling for read/write for each interface and specify higher processing priority

File: mh5_hardware/urdf/mh5_hardware.xacro (robot description, xacro)
@@ -5,11 +5,12 @@
       <param name="init_${name}">${address},${length},${value} </param>
     </xacro:macro>
-    <xacro:macro name="common_init" params="direction">
+    <xacro:macro name="common_init" params="direction offset max_voltage max_velocity">
       <xacro:register_init name="return_delay" address="9" length="1" value="0" />
       <xacro:register_init name="drive_mode" address="10" length="1" value="${direction}" />
       <xacro:register_init name="operating_mode" address="11" length="1" value="3" />
+      <xacro:register_init name="homing_offset" address="20" length="4" value="${offset}" />
       <xacro:register_init name="temp_limit" address="31" length="1" value="75" />
-      <xacro:register_init name="volt_limit" address="32" length="2" value="135" />
-      <xacro:register_init name="vel_limit" address="44" length="4" value="1023" />
+      <xacro:register_init name="volt_limit" address="32" length="2" value="${max_voltage}" />
+      <xacro:register_init name="vel_limit" address="44" length="4" value="${max_velocity}" />
       <xacro:register_init name="min_pos" address="52" length="4" value="0" />
       <xacro:register_init name="max_pos" address="48" length="4" value="4095" />
@@ -21,8 +22,9 @@
       <xacro:register_init name="indirect_led" address="178" length="2" value="65" />
     </xacro:macro>
-    <xacro:macro name="mh5_servo" params="joint_name id direction">
+    <xacro:macro name="xl430_servo" params="joint_name id direction offset=0">
       <joint name="${joint_name}">
         <param name="id">${id}</param>
-        <xacro:common_init direction="${direction}" />
+        <param name="model">XL430</param>
+        <xacro:common_init direction="${direction}" offset="${offset}" max_voltage="135" max_velocity="1023" />
         <state_interface name="position" />
         <state_interface name="velocity" />
@@ -39,5 +41,24 @@
       </joint>
     </xacro:macro>
-    <ros2_control name="upper_body" type="system" is_async="true" thread_priority="30">
+    <xacro:macro name="xl330_servo" params="joint_name id direction offset=0">
+      <joint name="${joint_name}">
+        <param name="id">${id}</param>
+        <param name="model">XL330</param>
+        <xacro:common_init direction="${direction}" offset="${offset}" max_voltage="70" max_velocity="445" />
+        <state_interface name="position" />
+        <state_interface name="velocity" />
+        <state_interface name="effort" />
+        <state_interface name="temperature" />
+        <state_interface name="voltage" />
+        <state_interface name="torque_enable" />
+        <state_interface name="error_overload" />
+        <state_interface name="error_electrical_shock" />
+        <state_interface name="error_motor_encoder" />
+        <state_interface name="error_overheating" />
+        <state_interface name="error_input_voltage" />
+        <state_interface name="led" />
+      </joint>
+    </xacro:macro>
+    <ros2_control name="upper_body" type="system" is_async="true" thread_priority="80">
       <xacro:if value="${use_mock_hardware}">
         <hardware>
@@ -57,14 +78,16 @@
         </hardware>
       </xacro:unless>
-      <xacro:mh5_servo joint_name="l_sho_p" id="34" direction="1" />
-      <xacro:mh5_servo joint_name="l_sho_r" id="33" direction="1" />
-      <xacro:mh5_servo joint_name="l_elb_r" id="32" direction="1" />
-      <xacro:mh5_servo joint_name="l_elb_p" id="31" direction="1" />
-      <xacro:mh5_servo joint_name="r_sho_p" id="44" direction="0" />
-      <xacro:mh5_servo joint_name="r_sho_r" id="43" direction="0" />
-      <xacro:mh5_servo joint_name="r_elb_r" id="42" direction="0" />
-      <xacro:mh5_servo joint_name="r_elb_p" id="41" direction="0" />
-      <xacro:mh5_servo joint_name="head_p" id="51" direction="0" />
-      <xacro:mh5_servo joint_name="head_y" id="52" direction="0" />
+      <xacro:xl430_servo joint_name="l_sho_p" id="34" direction="1" />
+      <xacro:xl430_servo joint_name="l_sho_r" id="33" direction="1" />
+      <xacro:xl430_servo joint_name="l_elb_r" id="32" direction="1" />
+      <xacro:xl430_servo joint_name="l_elb_p" id="31" direction="1" />
+      <xacro:xl330_servo joint_name="l_gripper" id="30" direction="0" />
+      <xacro:xl430_servo joint_name="r_sho_p" id="44" direction="0" />
+      <xacro:xl430_servo joint_name="r_sho_r" id="43" direction="0" />
+      <xacro:xl430_servo joint_name="r_elb_r" id="42" direction="0" />
+      <xacro:xl430_servo joint_name="r_elb_p" id="41" direction="0" />
+      <xacro:xl330_servo joint_name="r_gripper" id="40" direction="1" />
+      <xacro:xl430_servo joint_name="head_p" id="51" direction="0" />
+      <xacro:xl430_servo joint_name="head_y" id="52" direction="0" />
       <!-- <sensor name="pve_communication">
         <param name="rate">200</param>
@@ -73,5 +96,5 @@
       </sensor> -->
     </ros2_control>
-    <ros2_control name="lower_body" type="system"  is_async="true" thread_priority="30">
+    <ros2_control name="lower_body" type="system"  is_async="true" thread_priority="80">
       <xacro:if value="${use_mock_hardware}">
         <hardware>
@@ -91,16 +114,16 @@
         </hardware>
       </xacro:unless>
-      <xacro:mh5_servo joint_name="l_hip_r" id="16" direction="1" />
-      <xacro:mh5_servo joint_name="l_hip_p" id="15" direction="1" />
-      <xacro:mh5_servo joint_name="l_kne_p" id="14" direction="1" />   <!--  offset pi/2!  -->
-      <xacro:mh5_servo joint_name="l_kne_y" id="13" direction="1" />
-      <xacro:mh5_servo joint_name="l_ank_p" id="12" direction="1" />
-      <xacro:mh5_servo joint_name="l_ank_r" id="11" direction="0" />
-      <xacro:mh5_servo joint_name="r_hip_r" id="26" direction="0" />
-      <xacro:mh5_servo joint_name="r_hip_p" id="25" direction="1" />
-      <xacro:mh5_servo joint_name="r_kne_p" id="24" direction="1" />   <!--  offset pi/2!  -->
-      <xacro:mh5_servo joint_name="r_kne_y" id="23" direction="0" />
-      <xacro:mh5_servo joint_name="r_ank_p" id="22" direction="1" />
-      <xacro:mh5_servo joint_name="r_ank_r" id="21" direction="1" />
+      <xacro:xl430_servo joint_name="l_hip_r" id="16" direction="1" />
+      <xacro:xl430_servo joint_name="l_hip_p" id="15" direction="1" />
+      <xacro:xl430_servo joint_name="l_kne_p" id="14" direction="1" offset="-1024" />   <!--  offset pi/2!  -->
+      <xacro:xl430_servo joint_name="l_kne_y" id="13" direction="1" />
+      <xacro:xl430_servo joint_name="l_ank_p" id="12" direction="1" />
+      <xacro:xl430_servo joint_name="l_ank_r" id="11" direction="0" />
+      <xacro:xl430_servo joint_name="r_hip_r" id="26" direction="0" />
+      <xacro:xl430_servo joint_name="r_hip_p" id="25" direction="1" />
+      <xacro:xl430_servo joint_name="r_kne_p" id="24" direction="1" offset="-1024" />   <!--  offset pi/2!  -->
+      <xacro:xl430_servo joint_name="r_kne_y" id="23" direction="0" />
+      <xacro:xl430_servo joint_name="r_ank_p" id="22" direction="1" />
+      <xacro:xl430_servo joint_name="r_ank_r" id="21" direction="1" />
       <!-- <sensor name="pve_communication">
         <param name="rate">200</param>

Commit message: URDF updates - marco for servo simplification and added joint control

File: mh5_hardware/urdf/mh5_hardware.xacro (robot description, xacro)
@@ -23,9 +23,9 @@
       <xacro:register_init name="indirect_moving" address="180" length="2" value="122" />
     </xacro:macro>
-    <xacro:macro name="xl430_servo" params="joint_name id direction offset=0">
+    <xacro:macro name="servo" params="model joint_name id direction offset=0 max_voltage=135 max_velocity=1023">
       <joint name="${joint_name}">
         <param name="id">${id}</param>
-        <param name="model">XL430</param>
-        <xacro:common_init direction="${direction}" offset="${offset}" max_voltage="135" max_velocity="1023" />
+        <param name="model">${model}</param>
+        <xacro:common_init direction="${direction}" offset="${offset}" max_voltage="${max_voltage}" max_velocity="${max_velocity}" />
         <state_interface name="position" />
         <state_interface name="velocity" />
@@ -41,7 +41,8 @@
         <state_interface name="led" />
         <command_interface name ="torque_enable" />
+        <command_interface name="position" />
       </joint>
     </xacro:macro>
-    <xacro:macro name="xl330_servo" params="joint_name id direction offset=0">
+    <!-- <xacro:macro name="xl330_servo" params="joint_name id direction offset=0">
       <joint name="${joint_name}">
         <param name="id">${id}</param>
@@ -62,5 +63,5 @@
         <command_interface name ="torque_enable" />
       </joint>
-    </xacro:macro>
+    </xacro:macro> -->
     <ros2_control name="upper_body" type="system" is_async="true" thread_priority="80">
       <xacro:if value="${use_mock_hardware}">
@@ -83,16 +84,16 @@
         </hardware>
       </xacro:unless>
-      <xacro:xl430_servo joint_name="l_sho_p" id="34" direction="1" />
-      <xacro:xl430_servo joint_name="l_sho_r" id="33" direction="1" />
-      <xacro:xl430_servo joint_name="l_elb_r" id="32" direction="1" />
-      <xacro:xl430_servo joint_name="l_elb_p" id="31" direction="1" />
-      <xacro:xl330_servo joint_name="l_gripper" id="30" direction="0" />
-      <xacro:xl430_servo joint_name="r_sho_p" id="44" direction="0" />
-      <xacro:xl430_servo joint_name="r_sho_r" id="43" direction="0" />
-      <xacro:xl430_servo joint_name="r_elb_r" id="42" direction="0" />
-      <xacro:xl430_servo joint_name="r_elb_p" id="41" direction="0" />
-      <xacro:xl330_servo joint_name="r_gripper" id="40" direction="1" />
-      <xacro:xl430_servo joint_name="head_p" id="51" direction="0" />
-      <xacro:xl430_servo joint_name="head_y" id="52" direction="0" />
+      <xacro:servo model="XL430" joint_name="l_sho_p" id="34" direction="1" />
+      <xacro:servo model="XL430" joint_name="l_sho_r" id="33" direction="1" />
+      <xacro:servo model="XL430" joint_name="l_elb_r" id="32" direction="1" />
+      <xacro:servo model="XL430" joint_name="l_elb_p" id="31" direction="1" />
+      <xacro:servo model="XL330" joint_name="l_gripper" id="30" direction="0" max_voltage="70" max_velocity="445"/>
+      <xacro:servo model="XL430" joint_name="r_sho_p" id="44" direction="0" />
+      <xacro:servo model="XL430" joint_name="r_sho_r" id="43" direction="0" />
+      <xacro:servo model="XL430" joint_name="r_elb_r" id="42" direction="0" />
+      <xacro:servo model="XL430" joint_name="r_elb_p" id="41" direction="0" />
+      <xacro:servo model="XL330" joint_name="r_gripper" id="40" direction="1" max_voltage="70" max_velocity="445" />
+      <xacro:servo model="XL430" joint_name="head_p" id="51" direction="0" />
+      <xacro:servo model="XL430" joint_name="head_y" id="52" direction="0" />
       <!-- <sensor name="pve_communication">
         <param name="rate">200</param>
@@ -121,16 +122,16 @@
         </hardware>
       </xacro:unless>
-      <xacro:xl430_servo joint_name="l_hip_r" id="16" direction="1" />
-      <xacro:xl430_servo joint_name="l_hip_p" id="15" direction="1" />
-      <xacro:xl430_servo joint_name="l_kne_p" id="14" direction="1" offset="-1024" />   <!--  offset pi/2!  -->
-      <xacro:xl430_servo joint_name="l_kne_y" id="13" direction="1" />
-      <xacro:xl430_servo joint_name="l_ank_p" id="12" direction="1" />
-      <xacro:xl430_servo joint_name="l_ank_r" id="11" direction="0" />
-      <xacro:xl430_servo joint_name="r_hip_r" id="26" direction="0" />
-      <xacro:xl430_servo joint_name="r_hip_p" id="25" direction="1" />
-      <xacro:xl430_servo joint_name="r_kne_p" id="24" direction="1" offset="-1024" />   <!--  offset pi/2!  -->
-      <xacro:xl430_servo joint_name="r_kne_y" id="23" direction="0" />
-      <xacro:xl430_servo joint_name="r_ank_p" id="22" direction="1" />
-      <xacro:xl430_servo joint_name="r_ank_r" id="21" direction="1" />
+      <xacro:servo model="XL430" joint_name="l_hip_r" id="16" direction="1" />
+      <xacro:servo model="XL430" joint_name="l_hip_p" id="15" direction="1" />
+      <xacro:servo model="XL430" joint_name="l_kne_p" id="14" direction="1" offset="-1024" />   <!--  offset pi/2!  -->
+      <xacro:servo model="XL430" joint_name="l_kne_y" id="13" direction="1" />
+      <xacro:servo model="XL430" joint_name="l_ank_p" id="12" direction="1" />
+      <xacro:servo model="XL430" joint_name="l_ank_r" id="11" direction="0" />
+      <xacro:servo model="XL430" joint_name="r_hip_r" id="26" direction="0" />
+      <xacro:servo model="XL430" joint_name="r_hip_p" id="25" direction="1" />
+      <xacro:servo model="XL430" joint_name="r_kne_p" id="24" direction="1" offset="-1024" />   <!--  offset pi/2!  -->
+      <xacro:servo model="XL430" joint_name="r_kne_y" id="23" direction="0" />
+      <xacro:servo model="XL430" joint_name="r_ank_p" id="22" direction="1" />
+      <xacro:servo model="XL430" joint_name="r_ank_r" id="21" direction="1" />
       <!-- <sensor name="pve_communication">
         <param name="rate">200</param>
